Commit message: WIP: Modified URDF

File: controller_testing/urdf/testing.urdf.xacro (robot description, xacro)
@@ -29,4 +29,60 @@
     <child link="base_link" />
   </joint>
+  <joint name="thruster1_joint" type="continuous" ccw="true">
+    <origin rpy="-1.571 1.571 -0.785" xyz="0.14 -0.092 0.0" />
+    <parent link="base_link" />
+    <child link="thruster" />
+    <axis xyz="0 0 -1" />
+    <limits effort="-1" velocity="-1" />
+  </joint>
+  <joint name="thruster2_joint" type="continuous" ccw="true">
+    <origin rpy="-1.571 1.571 -2.356" xyz="0.14 0.092 0.0" />
+    <parent link="base_link" />
+    <child link="thruster" />
+    <axis xyz="0 0 -1" />
+    <limits effort="-1" velocity="-1" />
+  </joint>
+  <joint name="thruster3_joint" type="continuous" ccw="false">
+    <origin rpy="-1.571 1.571 0.785" xyz="-0.15 -0.092 0.0" />
+    <parent link="base_link" />
+    <child link="thruster" />
+    <axis xyz="0 0 -1" />
+    <limits effort="-1" velocity="-1" />
+  </joint>
+  <joint name="thruster4_joint" type="continuous" ccw="false">
+    <origin rpy="-1.571 1.571 2.356" xyz="-0.15 0.092 0.0" />
+    <parent link="base_link" />
+    <child link="thruster" />
+    <axis xyz="0 0 -1" />
+    <limits effort="-1" velocity="-1" />
+  </joint>
+  <joint name="thruster5_joint" type="continuous" ccw="true">
+    <origin rpy="0 0 0" xyz="0.118 -0.215 0.064" />
+    <parent link="base_link" />
+    <child link="thruster" />
+    <axis xyz="0 0 -1" />
+    <limits effort="-1" velocity="-1" />
+  </joint>
+  <joint name="thruster6_joint" type="continuous" ccw="false">
+    <origin rpy="0 0 0" xyz="0.118 0.215 0.064" />
+    <parent link="base_link" />
+    <child link="thruster" />
+    <axis xyz="0 0 -1" />
+    <limits effort="-1" velocity="-1" />
+  </joint>
+  <joint name="thruster7_joint" type="continuous" ccw="false">
+    <origin rpy="0 0 0" xyz="-0.118 -0.215 0.064" />
+    <parent link="base_link" />
+    <child link="thruster" />
+    <axis xyz="0 0 -1" />
+    <limits effort="-1" velocity="-1" />
+  </joint>
+  <joint name="thruster8_joint" type="continuous" ccw="true">
+    <origin rpy="0 0 0" xyz="-0.118 0.215 0.064" />
+    <parent link="base_link" />
+    <child link="thruster" />
+    <axis xyz="0 0 -1" />
+    <limits effort="-1" velocity="-1" />
+  </joint>
   <ros2_control name="testing" type="system">
     <hardware>
@@ -58,4 +114,28 @@
       <state_interface name="velocity" />
     </joint>
+    <joint name="thruster1_joint">
+      <command_interface name="effort" />
+    </joint>
+    <joint name="thruster2_joint">
+      <command_interface name="effort" />
+    </joint>
+    <joint name="thruster3_joint">
+      <command_interface name="effort" />
+    </joint>
+    <joint name="thruster4_joint">
+      <command_interface name="effort" />
+    </joint>
+    <joint name="thruster5_joint">
+      <command_interface name="effort" />
+    </joint>
+    <joint name="thruster6_joint">
+      <command_interface name="effort" />
+    </joint>
+    <joint name="thruster7_joint">
+      <command_interface name="effort" />
+    </joint>
+    <joint name="thruster8_joint">
+      <command_interface name="effort" />
+    </joint>
   </ros2_control>
 </robot>

Commit message: Partially works. Still need to fix TAM controller

File: controller_testing/urdf/testing.urdf.xacro (robot description, xacro)
@@ -29,59 +29,51 @@
     <child link="base_link" />
   </joint>
-  <joint name="thruster1_joint" type="continuous" ccw="true">
+  <joint name="thruster_1" type="continuous" ccw="true">
     <origin rpy="-1.571 1.571 -0.785" xyz="0.14 -0.092 0.0" />
     <parent link="base_link" />
-    <child link="thruster" />
+    <child link="thruster_1" />
     <axis xyz="0 0 -1" />
-    <limits effort="-1" velocity="-1" />
   </joint>
-  <joint name="thruster2_joint" type="continuous" ccw="true">
+  <joint name="thruster_2" type="continuous" ccw="true">
     <origin rpy="-1.571 1.571 -2.356" xyz="0.14 0.092 0.0" />
     <parent link="base_link" />
-    <child link="thruster" />
+    <child link="thruster_2" />
     <axis xyz="0 0 -1" />
-    <limits effort="-1" velocity="-1" />
   </joint>
-  <joint name="thruster3_joint" type="continuous" ccw="false">
+  <joint name="thruster_3" type="continuous" ccw="false">
     <origin rpy="-1.571 1.571 0.785" xyz="-0.15 -0.092 0.0" />
     <parent link="base_link" />
-    <child link="thruster" />
+    <child link="thruster_3" />
     <axis xyz="0 0 -1" />
-    <limits effort="-1" velocity="-1" />
   </joint>
-  <joint name="thruster4_joint" type="continuous" ccw="false">
+  <joint name="thruster_4" type="continuous" ccw="false">
     <origin rpy="-1.571 1.571 2.356" xyz="-0.15 0.092 0.0" />
     <parent link="base_link" />
-    <child link="thruster" />
+    <child link="thruster_4" />
     <axis xyz="0 0 -1" />
-    <limits effort="-1" velocity="-1" />
   </joint>
-  <joint name="thruster5_joint" type="continuous" ccw="true">
+  <joint name="thruster_5" type="continuous" ccw="true">
     <origin rpy="0 0 0" xyz="0.118 -0.215 0.064" />
     <parent link="base_link" />
-    <child link="thruster" />
+    <child link="thruster_5" />
     <axis xyz="0 0 -1" />
-    <limits effort="-1" velocity="-1" />
   </joint>
-  <joint name="thruster6_joint" type="continuous" ccw="false">
+  <joint name="thruster_6" type="continuous" ccw="false">
     <origin rpy="0 0 0" xyz="0.118 0.215 0.064" />
     <parent link="base_link" />
-    <child link="thruster" />
+    <child link="thruster_6" />
     <axis xyz="0 0 -1" />
-    <limits effort="-1" velocity="-1" />
   </joint>
-  <joint name="thruster7_joint" type="continuous" ccw="false">
+  <joint name="thruster_7" type="continuous" ccw="false">
     <origin rpy="0 0 0" xyz="-0.118 -0.215 0.064" />
     <parent link="base_link" />
-    <child link="thruster" />
+    <child link="thruster_7" />
     <axis xyz="0 0 -1" />
-    <limits effort="-1" velocity="-1" />
   </joint>
-  <joint name="thruster8_joint" type="continuous" ccw="true">
+  <joint name="thruster_8" type="continuous" ccw="true">
     <origin rpy="0 0 0" xyz="-0.118 0.215 0.064" />
     <parent link="base_link" />
-    <child link="thruster" />
+    <child link="thruster_8" />
     <axis xyz="0 0 -1" />
-    <limits effort="-1" velocity="-1" />
   </joint>
   <ros2_control name="testing" type="system">
@@ -114,27 +106,35 @@
       <state_interface name="velocity" />
     </joint>
-    <joint name="thruster1_joint">
-      <command_interface name="effort" />
+    <joint name="thruster_1">
+      <command_interface name="velocity" />
+      <state_interface name="velocity" />
     </joint>
-    <joint name="thruster2_joint">
-      <command_interface name="effort" />
+    <joint name="thruster_2">
+      <command_interface name="velocity" />
+      <state_interface name="velocity" />
     </joint>
-    <joint name="thruster3_joint">
-      <command_interface name="effort" />
+    <joint name="thruster_3">
+      <command_interface name="velocity" />
+      <state_interface name="velocity" />
     </joint>
-    <joint name="thruster4_joint">
-      <command_interface name="effort" />
+    <joint name="thruster_4">
+      <command_interface name="velocity" />
+      <state_interface name="velocity" />
     </joint>
-    <joint name="thruster5_joint">
-      <command_interface name="effort" />
+    <joint name="thruster_5">
+      <command_interface name="velocity" />
+      <state_interface name="velocity" />
     </joint>
-    <joint name="thruster6_joint">
-      <command_interface name="effort" />
+    <joint name="thruster_6">
+      <command_interface name="velocity" />
+      <state_interface name="velocity" />
     </joint>
-    <joint name="thruster7_joint">
-      <command_interface name="effort" />
+    <joint name="thruster_7">
+      <command_interface name="velocity" />
+      <state_interface name="velocity" />
     </joint>
-    <joint name="thruster8_joint">
-      <command_interface name="effort" />
+    <joint name="thruster_8">
+      <command_interface name="velocity" />
+      <state_interface name="velocity" />
     </joint>
   </ros2_control>

Commit message: Rewrite of tam controller and isolated bug in velocity controller

File: controller_testing/urdf/testing.urdf.xacro (robot description, xacro)
@@ -5,5 +5,8 @@
     <origin xyz="0 0 0" rpy="0 0 0" />
   </link>
-  <joint name="x" type="fixed">
+  <!-- Cartesian Joints -->
+  <!-- TODO(anyone): There is a weird thing going on right now with the cartesian joints and getting
+  the y joint loaded. Need to debug that. -->
+  <!-- <joint name="x" type="fixed">
     <parent link="base_footprint" />
     <child link="base_link" />
@@ -28,5 +31,6 @@
     <parent link="base_footprint" />
     <child link="base_link" />
-  </joint>
+  </joint> -->
+  <!-- Thruster joints -->
   <joint name="thruster_1" type="continuous" ccw="true">
     <origin rpy="-1.571 1.571 -0.785" xyz="0.14 -0.092 0.0" />
@@ -82,59 +86,45 @@
       <param name="calculate_dynamics">true</param>
     </hardware>
-    <joint name="x">
-      <command_interface name="effort" />
+    <!-- <joint name="x">
       <state_interface name="velocity" />
     </joint>
     <joint name="y">
-      <command_interface name="effort" />
       <state_interface name="velocity" />
     </joint>
     <joint name="z">
-      <command_interface name="effort" />
       <state_interface name="velocity" />
     </joint>
     <joint name="rx">
-      <command_interface name="effort" />
       <state_interface name="velocity" />
     </joint>
     <joint name="ry">
-      <command_interface name="effort" />
       <state_interface name="velocity" />
     </joint>
     <joint name="rz">
-      <command_interface name="effort" />
       <state_interface name="velocity" />
-    </joint>
+    </joint> -->
     <joint name="thruster_1">
       <command_interface name="velocity" />
-      <state_interface name="velocity" />
     </joint>
     <joint name="thruster_2">
       <command_interface name="velocity" />
-      <state_interface name="velocity" />
     </joint>
     <joint name="thruster_3">
       <command_interface name="velocity" />
-      <state_interface name="velocity" />
     </joint>
     <joint name="thruster_4">
       <command_interface name="velocity" />
-      <state_interface name="velocity" />
     </joint>
     <joint name="thruster_5">
       <command_interface name="velocity" />
-      <state_interface name="velocity" />
     </joint>
     <joint name="thruster_6">
       <command_interface name="velocity" />
-      <state_interface name="velocity" />
     </joint>
     <joint name="thruster_7">
       <command_interface name="velocity" />
-      <state_interface name="velocity" />
     </joint>
     <joint name="thruster_8">
       <command_interface name="velocity" />
-      <state_interface name="velocity" />
     </joint>
   </ros2_control>

Commit message: Cleaned up velocity controller and fixed some bugs

File: controller_testing/urdf/testing.urdf.xacro (robot description, xacro)
@@ -5,12 +5,34 @@
     <origin xyz="0 0 0" rpy="0 0 0" />
   </link>
+  <link name="thruster_1">
+    <origin xyz="0 0 0" rpy="0 0 0" />
+  </link>
+  <link name="thruster_2">
+    <origin xyz="0 0 0" rpy="0 0 0" />
+  </link>
+  <link name="thruster_3">
+    <origin xyz="0 0 0" rpy="0 0 0" />
+  </link>
+  <link name="thruster_4">
+    <origin xyz="0 0 0" rpy="0 0 0" />
+  </link>
+  <link name="thruster_5">
+    <origin xyz="0 0 0" rpy="0 0 0" />
+  </link>
+  <link name="thruster_6">
+    <origin xyz="0 0 0" rpy="0 0 0" />
+  </link>
+  <link name="thruster_7">
+    <origin xyz="0 0 0" rpy="0 0 0" />
+  </link>
+  <link name="thruster_8">
+    <origin xyz="0 0 0" rpy="0 0 0" />
+  </link>
   <!-- Cartesian Joints -->
-  <!-- TODO(anyone): There is a weird thing going on right now with the cartesian joints and getting
-  the y joint loaded. Need to debug that. -->
-  <!-- <joint name="x" type="fixed">
+  <joint name="x" type="fixed">
     <parent link="base_footprint" />
     <child link="base_link" />
   </joint>
-  <joint name="y" type="fixed">
+  <joint name="yo" type="fixed">
     <parent link="base_footprint" />
     <child link="base_link" />
@@ -31,5 +53,5 @@
     <parent link="base_footprint" />
     <child link="base_link" />
-  </joint> -->
+  </joint>
   <!-- Thruster joints -->
   <joint name="thruster_1" type="continuous" ccw="true">
@@ -86,22 +108,28 @@
       <param name="calculate_dynamics">true</param>
     </hardware>
-    <!-- <joint name="x">
+    <joint name="x">
       <state_interface name="velocity" />
+      <command_interface name="velocity" />
     </joint>
     <joint name="y">
       <state_interface name="velocity" />
+      <command_interface name="velocity" />
     </joint>
     <joint name="z">
       <state_interface name="velocity" />
+      <command_interface name="velocity" />
     </joint>
     <joint name="rx">
       <state_interface name="velocity" />
+      <command_interface name="velocity" />
     </joint>
     <joint name="ry">
       <state_interface name="velocity" />
+      <command_interface name="velocity" />
     </joint>
     <joint name="rz">
       <state_interface name="velocity" />
-    </joint> -->
+      <command_interface name="velocity" />
+    </joint>
     <joint name="thruster_1">
       <command_interface name="velocity" />

Commit message: Fixed bug with URDF and cleaned up thruster controller

File: controller_testing/urdf/testing.urdf.xacro (robot description, xacro)
@@ -34,5 +34,5 @@
     <child link="base_link" />
   </joint>
-  <joint name="yo" type="fixed">
+  <joint name="y" type="fixed">
     <parent link="base_footprint" />
     <child link="base_link" />
@@ -55,5 +55,5 @@
   </joint>
   <!-- Thruster joints -->
-  <joint name="thruster_1" type="continuous" ccw="true">
+  <joint name="thruster_1_joint" type="continuous" ccw="true">
     <origin rpy="-1.571 1.571 -0.785" xyz="0.14 -0.092 0.0" />
     <parent link="base_link" />
@@ -61,5 +61,5 @@
     <axis xyz="0 0 -1" />
   </joint>
-  <joint name="thruster_2" type="continuous" ccw="true">
+  <joint name="thruster_2_joint" type="continuous" ccw="true">
     <origin rpy="-1.571 1.571 -2.356" xyz="0.14 0.092 0.0" />
     <parent link="base_link" />
@@ -67,5 +67,5 @@
     <axis xyz="0 0 -1" />
   </joint>
-  <joint name="thruster_3" type="continuous" ccw="false">
+  <joint name="thruster_3_joint" type="continuous" ccw="false">
     <origin rpy="-1.571 1.571 0.785" xyz="-0.15 -0.092 0.0" />
     <parent link="base_link" />
@@ -73,5 +73,5 @@
     <axis xyz="0 0 -1" />
   </joint>
-  <joint name="thruster_4" type="continuous" ccw="false">
+  <joint name="thruster_4_joint" type="continuous" ccw="false">
     <origin rpy="-1.571 1.571 2.356" xyz="-0.15 0.092 0.0" />
     <parent link="base_link" />
@@ -79,5 +79,5 @@
     <axis xyz="0 0 -1" />
   </joint>
-  <joint name="thruster_5" type="continuous" ccw="true">
+  <joint name="thruster_5_joint" type="continuous" ccw="true">
     <origin rpy="0 0 0" xyz="0.118 -0.215 0.064" />
     <parent link="base_link" />
@@ -85,5 +85,5 @@
     <axis xyz="0 0 -1" />
   </joint>
-  <joint name="thruster_6" type="continuous" ccw="false">
+  <joint name="thruster_6_joint" type="continuous" ccw="false">
     <origin rpy="0 0 0" xyz="0.118 0.215 0.064" />
     <parent link="base_link" />
@@ -91,5 +91,5 @@
     <axis xyz="0 0 -1" />
   </joint>
-  <joint name="thruster_7" type="continuous" ccw="false">
+  <joint name="thruster_7_joint" type="continuous" ccw="false">
     <origin rpy="0 0 0" xyz="-0.118 -0.215 0.064" />
     <parent link="base_link" />
@@ -97,5 +97,5 @@
     <axis xyz="0 0 -1" />
   </joint>
-  <joint name="thruster_8" type="continuous" ccw="true">
+  <joint name="thruster_8_joint" type="continuous" ccw="true">
     <origin rpy="0 0 0" xyz="-0.118 0.215 0.064" />
     <parent link="base_link" />
@@ -106,52 +106,58 @@
     <hardware>
       <plugin>mock_components/GenericSystem</plugin>
-      <param name="calculate_dynamics">true</param>
+      <param name="calculate_dynamics">false</param>
     </hardware>
     <joint name="x">
-      <state_interface name="velocity" />
+      <state_interface name="velocity">
+        <param name="initial_value">0.0</param>
+      </state_interface>
+    </joint>
+    <joint name="y">
+      <state_interface name="velocity">
+        <param name="initial_value">0.0</param>
+      </state_interface>
+    </joint>
+    <joint name="z">
+      <state_interface name="velocity">
+        <param name="initial_value">0.0</param>
+      </state_interface>
+    </joint>
+    <joint name="rx">
+      <state_interface name="velocity">
+        <param name="initial_value">0.0</param>
+      </state_interface>
+    </joint>
+    <joint name="ry">
+      <state_interface name="velocity">
+        <param name="initial_value">0.0</param>
+      </state_interface>
+    </joint>
+    <joint name="rz">
+      <state_interface name="velocity">
+        <param name="initial_value">0.0</param>
+      </state_interface>
+    </joint>
+    <joint name="thruster_1_joint">
       <command_interface name="velocity" />
     </joint>
-    <joint name="y">
-      <state_interface name="velocity" />
+    <joint name="thruster_2_joint">
       <command_interface name="velocity" />
     </joint>
-    <joint name="z">
-      <state_interface name="velocity" />
+    <joint name="thruster_3_joint">
       <command_interface name="velocity" />
     </joint>
-    <joint name="rx">
-      <state_interface name="velocity" />
+    <joint name="thruster_4_joint">
       <command_interface name="velocity" />
     </joint>
-    <joint name="ry">
-      <state_interface name="velocity" />
+    <joint name="thruster_5_joint">
       <command_interface name="velocity" />
     </joint>
-    <joint name="rz">
-      <state_interface name="velocity" />
+    <joint name="thruster_6_joint">
       <command_interface name="velocity" />
     </joint>
-    <joint name="thruster_1">
+    <joint name="thruster_7_joint">
       <command_interface name="velocity" />
     </joint>
-    <joint name="thruster_2">
-      <command_interface name="velocity" />
-    </joint>
-    <joint name="thruster_3">
-      <command_interface name="velocity" />
-    </joint>
-    <joint name="thruster_4">
-      <command_interface name="velocity" />
-    </joint>
-    <joint name="thruster_5">
-      <command_interface name="velocity" />
-    </joint>
-    <joint name="thruster_6">
-      <command_interface name="velocity" />
-    </joint>
-    <joint name="thruster_7">
-      <command_interface name="velocity" />
-    </joint>
-    <joint name="thruster_8">
+    <joint name="thruster_8_joint">
       <command_interface name="velocity" />
     </joint>
