Commit message: Updated dockerfile and devcontainer

File: auv_control_demos/chained_controllers/xacro/chained_config.xacro (robot description, xacro)
@@ -1,4 +1,5 @@
 <?xml version="1.0"?>
-<robot name="auv" xmlns:xacro="http://ros.org/wiki/xacro">
+<robot name="auv"
+       xmlns:xacro="http://ros.org/wiki/xacro">
   <xacro:include filename="$(find auv_control_demos)/xacro/chained_urdf.xacro" />
   <xacro:include filename="$(find auv_control_demos)/xacro/chained_ros2_control.xacro" />

File: auv_control_demos/chained_controllers/xacro/chained_ros2_control.xacro (robot description, xacro)
@@ -1,5 +1,6 @@
 <?xml version="1.0"?>
 <robot xmlns:xacro="http://www.ros.org/wiki/xacro">
-  <ros2_control name="demo_hardware" type="system">
+  <ros2_control name="demo_hardware"
+                type="system">
     <hardware>
       <plugin>mock_components/GenericSystem</plugin>

File: auv_control_demos/chained_controllers/xacro/chained_urdf.xacro (robot description, xacro)
@@ -1,102 +1,142 @@
 <?xml version="1.0"?>
-<robot xmlns:xacro="http://www.ros.org/wiki/xacro" name="auv">
+<robot xmlns:xacro="http://www.ros.org/wiki/xacro"
+       name="auv">
   <link name="base_footprint" />
   <link name="base_link">
-    <origin xyz="0 0 0" rpy="0 0 0" />
+    <origin xyz="0 0 0"
+            rpy="0 0 0" />
   </link>
   <link name="thruster_1">
-    <origin xyz="0 0 0" rpy="0 0 0" />
+    <origin xyz="0 0 0"
+            rpy="0 0 0" />
   </link>
   <link name="thruster_2">
-    <origin xyz="0 0 0" rpy="0 0 0" />
+    <origin xyz="0 0 0"
+            rpy="0 0 0" />
   </link>
   <link name="thruster_3">
-    <origin xyz="0 0 0" rpy="0 0 0" />
+    <origin xyz="0 0 0"
+            rpy="0 0 0" />
   </link>
   <link name="thruster_4">
-    <origin xyz="0 0 0" rpy="0 0 0" />
+    <origin xyz="0 0 0"
+            rpy="0 0 0" />
   </link>
   <link name="thruster_5">
-    <origin xyz="0 0 0" rpy="0 0 0" />
+    <origin xyz="0 0 0"
+            rpy="0 0 0" />
   </link>
   <link name="thruster_6">
-    <origin xyz="0 0 0" rpy="0 0 0" />
+    <origin xyz="0 0 0"
+            rpy="0 0 0" />
   </link>
   <link name="thruster_7">
-    <origin xyz="0 0 0" rpy="0 0 0" />
+    <origin xyz="0 0 0"
+            rpy="0 0 0" />
   </link>
   <link name="thruster_8">
-    <origin xyz="0 0 0" rpy="0 0 0" />
+    <origin xyz="0 0 0"
+            rpy="0 0 0" />
   </link>
   <!-- Cartesian Joints -->
-  <joint name="x" type="fixed">
+  <joint name="x"
+         type="fixed">
     <parent link="base_footprint" />
     <child link="base_link" />
   </joint>
-  <joint name="y" type="fixed">
+  <joint name="y"
+         type="fixed">
     <parent link="base_footprint" />
     <child link="base_link" />
   </joint>
-  <joint name="z" type="fixed">
+  <joint name="z"
+         type="fixed">
     <parent link="base_footprint" />
     <child link="base_link" />
   </joint>
-  <joint name="rx" type="fixed">
+  <joint name="rx"
+         type="fixed">
     <parent link="base_footprint" />
     <child link="base_link" />
   </joint>
-  <joint name="ry" type="fixed">
+  <joint name="ry"
+         type="fixed">
     <parent link="base_footprint" />
     <child link="base_link" />
   </joint>
-  <joint name="rz" type="fixed">
+  <joint name="rz"
+         type="fixed">
     <parent link="base_footprint" />
     <child link="base_link" />
   </joint>
   <!-- Thruster joints -->
-  <joint name="thruster_1_joint" type="continuous" ccw="true">
-    <origin rpy="-1.571 1.571 -0.785" xyz="0.14 -0.092 0.0" />
+  <joint name="thruster_1_joint"
+         type="continuous"
+         ccw="true">
+    <origin rpy="-1.571 1.571 -0.785"
+            xyz="0.14 -0.092 0.0" />
     <parent link="base_link" />
     <child link="thruster_1" />
     <axis xyz="0 0 -1" />
   </joint>
-  <joint name="thruster_2_joint" type="continuous" ccw="true">
-    <origin rpy="-1.571 1.571 -2.356" xyz="0.14 0.092 0.0" />
+  <joint name="thruster_2_joint"
+         type="continuous"
+         ccw="true">
+    <origin rpy="-1.571 1.571 -2.356"
+            xyz="0.14 0.092 0.0" />
     <parent link="base_link" />
     <child link="thruster_2" />
     <axis xyz="0 0 -1" />
   </joint>
-  <joint name="thruster_3_joint" type="continuous" ccw="false">
-    <origin rpy="-1.571 1.571 0.785" xyz="-0.15 -0.092 0.0" />
+  <joint name="thruster_3_joint"
+         type="continuous"
+         ccw="false">
+    <origin rpy="-1.571 1.571 0.785"
+            xyz="-0.15 -0.092 0.0" />
     <parent link="base_link" />
     <child link="thruster_3" />
     <axis xyz="0 0 -1" />
   </joint>
-  <joint name="thruster_4_joint" type="continuous" ccw="false">
-    <origin rpy="-1.571 1.571 2.356" xyz="-0.15 0.092 0.0" />
+  <joint name="thruster_4_joint"
+         type="continuous"
+         ccw="false">
+    <origin rpy="-1.571 1.571 2.356"
+            xyz="-0.15 0.092 0.0" />
     <parent link="base_link" />
     <child link="thruster_4" />
     <axis xyz="0 0 -1" />
   </joint>
-  <joint name="thruster_5_joint" type="continuous" ccw="true">
-    <origin rpy="0 0 0" xyz="0.118 -0.215 0.064" />
+  <joint name="thruster_5_joint"
+         type="continuous"
+         ccw="true">
+    <origin rpy="0 0 0"
+            xyz="0.118 -0.215 0.064" />
     <parent link="base_link" />
     <child link="thruster_5" />
     <axis xyz="0 0 -1" />
   </joint>
-  <joint name="thruster_6_joint" type="continuous" ccw="false">
-    <origin rpy="0 0 0" xyz="0.118 0.215 0.064" />
+  <joint name="thruster_6_joint"
+         type="continuous"
+         ccw="false">
+    <origin rpy="0 0 0"
+            xyz="0.118 0.215 0.064" />
     <parent link="base_link" />
     <child link="thruster_6" />
     <axis xyz="0 0 -1" />
   </joint>
-  <joint name="thruster_7_joint" type="continuous" ccw="false">
-    <origin rpy="0 0 0" xyz="-0.118 -0.215 0.064" />
+  <joint name="thruster_7_joint"
+         type="continuous"
+         ccw="false">
+    <origin rpy="0 0 0"
+            xyz="-0.118 -0.215 0.064" />
     <parent link="base_link" />
     <child link="thruster_7" />
     <axis xyz="0 0 -1" />
   </joint>
-  <joint name="thruster_8_joint" type="continuous" ccw="true">
-    <origin rpy="0 0 0" xyz="-0.118 0.215 0.064" />
+  <joint name="thruster_8_joint"
+         type="continuous"
+         ccw="true">
+    <origin rpy="0 0 0"
+            xyz="-0.118 0.215 0.064" />
     <parent link="base_link" />
     <child link="thruster_8" />

File: auv_control_demos/individual_controller/xacro/individual_config.xacro (robot description, xacro)
@@ -1,4 +1,5 @@
 <?xml version="1.0"?>
-<robot name="auv" xmlns:xacro="http://ros.org/wiki/xacro">
+<robot name="auv"
+       xmlns:xacro="http://ros.org/wiki/xacro">
   <xacro:include filename="$(find auv_control_demos)/xacro/individual_urdf.xacro" />
   <xacro:include filename="$(find auv_control_demos)/xacro/individual_ros2_control.xacro" />

File: auv_control_demos/individual_controller/xacro/individual_ros2_control.xacro (robot description, xacro)
@@ -1,5 +1,7 @@
 <?xml version="1.0"?>
-<robot xmlns:xacro="http://www.ros.org/wiki/xacro" name="control">
-  <ros2_control name="demo_hardware" type="system">
+<robot xmlns:xacro="http://www.ros.org/wiki/xacro"
+       name="control">
+  <ros2_control name="demo_hardware"
+                type="system">
     <hardware>
       <plugin>mock_components/GenericSystem</plugin>

File: auv_control_demos/individual_controller/xacro/individual_urdf.xacro (robot description, xacro)
@@ -1,32 +1,40 @@
 <?xml version="1.0"?>
-<robot xmlns:xacro="http://www.ros.org/wiki/xacro" name="auv">
-    <link name="base_footprint" />
-    <link name="base_link">
-      <origin xyz="0 0 0" rpy="0 0 0" />
-    </link>
-    <!-- Cartesian Joints -->
-    <joint name="x" type="fixed">
-      <parent link="base_footprint" />
-      <child link="base_link" />
-    </joint>
-    <joint name="y" type="fixed">
-      <parent link="base_footprint" />
-      <child link="base_link" />
-    </joint>
-    <joint name="z" type="fixed">
-      <parent link="base_footprint" />
-      <child link="base_link" />
-    </joint>
-    <joint name="rx" type="fixed">
-      <parent link="base_footprint" />
-      <child link="base_link" />
-    </joint>
-    <joint name="ry" type="fixed">
-      <parent link="base_footprint" />
-      <child link="base_link" />
-    </joint>
-    <joint name="rz" type="fixed">
-      <parent link="base_footprint" />
-      <child link="base_link" />
-    </joint>
+<robot xmlns:xacro="http://www.ros.org/wiki/xacro"
+       name="auv">
+  <link name="base_footprint" />
+  <link name="base_link">
+    <origin xyz="0 0 0"
+            rpy="0 0 0" />
+  </link>
+  <!-- Cartesian Joints -->
+  <joint name="x"
+         type="fixed">
+    <parent link="base_footprint" />
+    <child link="base_link" />
+  </joint>
+  <joint name="y"
+         type="fixed">
+    <parent link="base_footprint" />
+    <child link="base_link" />
+  </joint>
+  <joint name="z"
+         type="fixed">
+    <parent link="base_footprint" />
+    <child link="base_link" />
+  </joint>
+  <joint name="rx"
+         type="fixed">
+    <parent link="base_footprint" />
+    <child link="base_link" />
+  </joint>
+  <joint name="ry"
+         type="fixed">
+    <parent link="base_footprint" />
+    <child link="base_link" />
+  </joint>
+  <joint name="rz"
+         type="fixed">
+    <parent link="base_footprint" />
+    <child link="base_link" />
+  </joint>
 </robot>
