Commit message: Updates to support ROS 2 Rolling (#41)
* Updated dockerfile and devcontainer

* Cleanup controllers for latest version of ros2_control

* Removed dll_export stuff

* Cleanup devcontainer

* Updated to use latest version of hydrodynamics

* Fix clang tidy errors

* Resolve final error in CI

* Fixed dev container name

File: auv_control_demos/chained_controllers/xacro/chained_urdf.xacro (robot description, xacro)
@@ -1,105 +1,145 @@
 <?xml version="1.0"?>
-<robot xmlns:xacro="http://www.ros.org/wiki/xacro" name="auv">
-  <link name="base_footprint" />
-  <link name="base_link">
-    <origin xyz="0 0 0" rpy="0 0 0" />
-  </link>
-  <link name="thruster_1">
-    <origin xyz="0 0 0" rpy="0 0 0" />
-  </link>
-  <link name="thruster_2">
-    <origin xyz="0 0 0" rpy="0 0 0" />
-  </link>
-  <link name="thruster_3">
-    <origin xyz="0 0 0" rpy="0 0 0" />
-  </link>
-  <link name="thruster_4">
-    <origin xyz="0 0 0" rpy="0 0 0" />
-  </link>
-  <link name="thruster_5">
-    <origin xyz="0 0 0" rpy="0 0 0" />
-  </link>
-  <link name="thruster_6">
-    <origin xyz="0 0 0" rpy="0 0 0" />
-  </link>
-  <link name="thruster_7">
-    <origin xyz="0 0 0" rpy="0 0 0" />
-  </link>
-  <link name="thruster_8">
-    <origin xyz="0 0 0" rpy="0 0 0" />
-  </link>
-  <!-- Cartesian Joints -->
-  <joint name="x" type="fixed">
-    <parent link="base_footprint" />
-    <child link="base_link" />
-  </joint>
-  <joint name="y" type="fixed">
-    <parent link="base_footprint" />
-    <child link="base_link" />
-  </joint>
-  <joint name="z" type="fixed">
-    <parent link="base_footprint" />
-    <child link="base_link" />
-  </joint>
-  <joint name="rx" type="fixed">
-    <parent link="base_footprint" />
-    <child link="base_link" />
-  </joint>
-  <joint name="ry" type="fixed">
-    <parent link="base_footprint" />
-    <child link="base_link" />
-  </joint>
-  <joint name="rz" type="fixed">
-    <parent link="base_footprint" />
-    <child link="base_link" />
-  </joint>
-  <!-- Thruster joints -->
-  <joint name="thruster_1_joint" type="continuous" ccw="true">
-    <origin rpy="-1.571 1.571 -0.785" xyz="0.14 -0.092 0.0" />
-    <parent link="base_link" />
-    <child link="thruster_1" />
-    <axis xyz="0 0 -1" />
-  </joint>
-  <joint name="thruster_2_joint" type="continuous" ccw="true">
-    <origin rpy="-1.571 1.571 -2.356" xyz="0.14 0.092 0.0" />
-    <parent link="base_link" />
-    <child link="thruster_2" />
-    <axis xyz="0 0 -1" />
-  </joint>
-  <joint name="thruster_3_joint" type="continuous" ccw="false">
-    <origin rpy="-1.571 1.571 0.785" xyz="-0.15 -0.092 0.0" />
-    <parent link="base_link" />
-    <child link="thruster_3" />
-    <axis xyz="0 0 -1" />
-  </joint>
-  <joint name="thruster_4_joint" type="continuous" ccw="false">
-    <origin rpy="-1.571 1.571 2.356" xyz="-0.15 0.092 0.0" />
-    <parent link="base_link" />
-    <child link="thruster_4" />
-    <axis xyz="0 0 -1" />
-  </joint>
-  <joint name="thruster_5_joint" type="continuous" ccw="true">
-    <origin rpy="0 0 0" xyz="0.118 -0.215 0.064" />
-    <parent link="base_link" />
-    <child link="thruster_5" />
-    <axis xyz="0 0 -1" />
-  </joint>
-  <joint name="thruster_6_joint" type="continuous" ccw="false">
-    <origin rpy="0 0 0" xyz="0.118 0.215 0.064" />
-    <parent link="base_link" />
-    <child link="thruster_6" />
-    <axis xyz="0 0 -1" />
-  </joint>
-  <joint name="thruster_7_joint" type="continuous" ccw="false">
-    <origin rpy="0 0 0" xyz="-0.118 -0.215 0.064" />
-    <parent link="base_link" />
-    <child link="thruster_7" />
-    <axis xyz="0 0 -1" />
-  </joint>
-  <joint name="thruster_8_joint" type="continuous" ccw="true">
-    <origin rpy="0 0 0" xyz="-0.118 0.215 0.064" />
-    <parent link="base_link" />
-    <child link="thruster_8" />
-    <axis xyz="0 0 -1" />
-  </joint>
+<robot xmlns:xacro="http://www.ros.org/wiki/xacro"
+       name="auv">
+        <link name="odom" />
+        <link name="base_link">
+                <origin xyz="0 0 0"
+                        rpy="0 0 0" />
+        </link>
+        <link name="thruster_1">
+                <origin xyz="0 0 0"
+                        rpy="0 0 0" />
+        </link>
+        <link name="thruster_2">
+                <origin xyz="0 0 0"
+                        rpy="0 0 0" />
+        </link>
+        <link name="thruster_3">
+                <origin xyz="0 0 0"
+                        rpy="0 0 0" />
+        </link>
+        <link name="thruster_4">
+                <origin xyz="0 0 0"
+                        rpy="0 0 0" />
+        </link>
+        <link name="thruster_5">
+                <origin xyz="0 0 0"
+                        rpy="0 0 0" />
+        </link>
+        <link name="thruster_6">
+                <origin xyz="0 0 0"
+                        rpy="0 0 0" />
+        </link>
+        <link name="thruster_7">
+                <origin xyz="0 0 0"
+                        rpy="0 0 0" />
+        </link>
+        <link name="thruster_8">
+                <origin xyz="0 0 0"
+                        rpy="0 0 0" />
+        </link>
+        <!-- Cartesian Joints -->
+        <joint name="x"
+               type="continuous">
+                <parent link="odom" />
+                <child link="base_link" />
+        </joint>
+        <joint name="y"
+               type="continuous">
+                <parent link="odom" />
+                <child link="base_link" />
+        </joint>
+        <joint name="z"
+               type="continuous">
+                <parent link="odom" />
+                <child link="base_link" />
+        </joint>
+        <joint name="rx"
+               type="continuous">
+                <parent link="odom" />
+                <child link="base_link" />
+        </joint>
+        <joint name="ry"
+               type="continuous">
+                <parent link="odom" />
+                <child link="base_link" />
+        </joint>
+        <joint name="rz"
+               type="continuous">
+                <parent link="odom" />
+                <child link="base_link" />
+        </joint>
+        <!-- Thruster joints -->
+        <joint name="thruster_1_joint"
+               type="continuous"
+               ccw="true">
+                <origin rpy="-1.571 1.571 -0.785"
+                        xyz="0.14 -0.092 0.0" />
+                <parent link="base_link" />
+                <child link="thruster_1" />
+                <axis xyz="0 0 -1" />
+        </joint>
+        <joint name="thruster_2_joint"
+               type="continuous"
+               ccw="true">
+                <origin rpy="-1.571 1.571 -2.356"
+                        xyz="0.14 0.092 0.0" />
+                <parent link="base_link" />
+                <child link="thruster_2" />
+                <axis xyz="0 0 -1" />
+        </joint>
+        <joint name="thruster_3_joint"
+               type="continuous"
+               ccw="false">
+                <origin rpy="-1.571 1.571 0.785"
+                        xyz="-0.15 -0.092 0.0" />
+                <parent link="base_link" />
+                <child link="thruster_3" />
+                <axis xyz="0 0 -1" />
+        </joint>
+        <joint name="thruster_4_joint"
+               type="continuous"
+               ccw="false">
+                <origin rpy="-1.571 1.571 2.356"
+                        xyz="-0.15 0.092 0.0" />
+                <parent link="base_link" />
+                <child link="thruster_4" />
+                <axis xyz="0 0 -1" />
+        </joint>
+        <joint name="thruster_5_joint"
+               type="continuous"
+               ccw="true">
+                <origin rpy="0 0 0"
+                        xyz="0.118 -0.215 0.064" />
+                <parent link="base_link" />
+                <child link="thruster_5" />
+                <axis xyz="0 0 -1" />
+        </joint>
+        <joint name="thruster_6_joint"
+               type="continuous"
+               ccw="false">
+                <origin rpy="0 0 0"
+                        xyz="0.118 0.215 0.064" />
+                <parent link="base_link" />
+                <child link="thruster_6" />
+                <axis xyz="0 0 -1" />
+        </joint>
+        <joint name="thruster_7_joint"
+               type="continuous"
+               ccw="false">
+                <origin rpy="0 0 0"
+                        xyz="-0.118 -0.215 0.064" />
+                <parent link="base_link" />
+                <child link="thruster_7" />
+                <axis xyz="0 0 -1" />
+        </joint>
+        <joint name="thruster_8_joint"
+               type="continuous"
+               ccw="true">
+                <origin rpy="0 0 0"
+                        xyz="-0.118 0.215 0.064" />
+                <parent link="base_link" />
+                <child link="thruster_8" />
+                <axis xyz="0 0 -1" />
+        </joint>
 </robot>

File: auv_control_demos/individual_controller/xacro/individual_urdf.xacro (robot description, xacro)
@@ -1,32 +1,40 @@
 <?xml version="1.0"?>
-<robot xmlns:xacro="http://www.ros.org/wiki/xacro" name="auv">
-    <link name="base_footprint" />
-    <link name="base_link">
-      <origin xyz="0 0 0" rpy="0 0 0" />
-    </link>
-    <!-- Cartesian Joints -->
-    <joint name="x" type="fixed">
-      <parent link="base_footprint" />
-      <child link="base_link" />
-    </joint>
-    <joint name="y" type="fixed">
-      <parent link="base_footprint" />
-      <child link="base_link" />
-    </joint>
-    <joint name="z" type="fixed">
-      <parent link="base_footprint" />
-      <child link="base_link" />
-    </joint>
-    <joint name="rx" type="fixed">
-      <parent link="base_footprint" />
-      <child link="base_link" />
-    </joint>
-    <joint name="ry" type="fixed">
-      <parent link="base_footprint" />
-      <child link="base_link" />
-    </joint>
-    <joint name="rz" type="fixed">
-      <parent link="base_footprint" />
-      <child link="base_link" />
-    </joint>
+<robot xmlns:xacro="http://www.ros.org/wiki/xacro"
+       name="auv">
+  <link name="odom" />
+  <link name="base_link">
+    <origin xyz="0 0 0"
+            rpy="0 0 0" />
+  </link>
+  <!-- Cartesian Joints -->
+  <joint name="x"
+         type="continuous">
+    <parent link="odom" />
+    <child link="base_link" />
+  </joint>
+  <joint name="y"
+         type="continuous">
+    <parent link="odom" />
+    <child link="base_link" />
+  </joint>
+  <joint name="z"
+         type="continuous">
+    <parent link="odom" />
+    <child link="base_link" />
+  </joint>
+  <joint name="rx"
+         type="continuous">
+    <parent link="odom" />
+    <child link="base_link" />
+  </joint>
+  <joint name="ry"
+         type="continuous">
+    <parent link="odom" />
+    <child link="base_link" />
+  </joint>
+  <joint name="rz"
+         type="continuous">
+    <parent link="odom" />
+    <child link="base_link" />
+  </joint>
 </robot>
