Commit message: Fixed stale demos

File: auv_control_demos/chained_controllers/xacro/chained.ros2_control.xacro (robot description, xacro)
@@ -7,34 +7,4 @@
       <param name="calculate_dynamics">false</param>
     </hardware>
-    <joint name="x">
-      <state_interface name="velocity">
-        <param name="initial_value">0.0</param>
-      </state_interface>
-    </joint>
-    <joint name="y">
-      <state_interface name="velocity">
-        <param name="initial_value">0.0</param>
-      </state_interface>
-    </joint>
-    <joint name="z">
-      <state_interface name="velocity">
-        <param name="initial_value">0.0</param>
-      </state_interface>
-    </joint>
-    <joint name="rx">
-      <state_interface name="velocity">
-        <param name="initial_value">0.0</param>
-      </state_interface>
-    </joint>
-    <joint name="ry">
-      <state_interface name="velocity">
-        <param name="initial_value">0.0</param>
-      </state_interface>
-    </joint>
-    <joint name="rz">
-      <state_interface name="velocity">
-        <param name="initial_value">0.0</param>
-      </state_interface>
-    </joint>
     <joint name="thruster_1_joint">
       <command_interface name="pwm" />
