Commit message: solver compile working

File: output.urdf (robot description, URDF)
Before this commit: robot bluerov2_heavy, 4 links, 3 joints
Links:
- added link manipulator_base_link, mass 0.0001
- added link manipulator_link, mass 0.0001
Joints:
- added joint axis_d: type revolute, parent manipulator_base_link, child manipulator_link, origin xyz=-0.02 0 0.033, axis 0 1 0, limit lower=-3.49 upper=3.49 effort=9.0 velocity=0.5
- added joint manipulator_base_joint: type fixed, parent base_link, child manipulator_base_link, origin xyz=0.01 -0.01 0.01 rpy=0 0 0

Commit message: test full urdf and start debugging tpik controller

File: output.urdf (robot description, URDF)
Before this commit: robot bluerov2_heavy, 6 links, 5 joints
Links:
- removed link manipulator_base_link
- removed link manipulator_link
- added link alpha_base_link, mass 0.0001; collision cylinder length=0.150 radius=0.020; visual mesh filename=file:///home/ubuntu/ws_blue/install/reach_description/share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
- added link alpha_m1_link, mass 0.200; collision cylinder length=0.1 radius=0.020; visual mesh filename=file:///home/ubuntu/ws_blue/install/reach_description/share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
- added link alpha_m2_1_1_link, mass 0.194; collision cylinder length=0.033 radius=0.020; visual mesh filename=file:///home/ubuntu/ws_blue/install/reach_description/share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
- added link alpha_m2_1_3_link, mass 0.115; collision cylinder length=0.033 radius=0.020; visual mesh filename=file:///home/ubuntu/ws_blue/install/reach_description/share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
- added link alpha_m2_link, mass 0.429; collision cylinder length=0.040 radius=0.020; collision cylinder length=0.040 radius=0.020
- added link alpha_m3_inline_link, mass 0.341; collision cylinder length=0.150 radius=0.020; visual mesh filename=file:///home/ubuntu/ws_blue/install/reach_description/share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
- added link alpha_push_rod, mass 0.0001; visual box size=0.001 0.001 0.001
- added link alpha_rs1_124_link, mass 0.0001; collision cylinder length=0.1 radius=0.020; visual mesh filename=file:///home/ubuntu/ws_blue/install/reach_description/share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
- added link alpha_rs1_130_link, mass 0.055; collision box size=0.012 0.03 0.09; visual mesh filename=file:///home/ubuntu/ws_blue/install/reach_description/share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
- added link alpha_rs1_139_link, mass 0.055; collision box size=0.012 0.03 0.09; visual mesh filename=file:///home/ubuntu/ws_blue/install/reach_description/share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
- added link alpha_tcp, mass 0.0001
- added link float_link; collision box size=0.2285 0.2875 0.005; collision box size=0.2285 0.2875 0.015
- added link mount_link
- link base_link: geometry collision box size=0.457 0.575 0.05; visual mesh filename=file:///home/ubuntu/ws_blue/install/blue_description/share/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 scale=0.025 0.025 0.025
Joints:
- removed joint axis_d
- removed joint manipulator_base_joint
- added joint alpha_axis_a: type prismatic, parent alpha_rs1_124_link, child alpha_push_rod, origin xyz=0 0 0.009 rpy=0 0 0, axis 0 0 1, limit lower=0 upper=0.015 effort=10 velocity=10
- added joint alpha_axis_b: type revolute, parent alpha_m2_1_3_link, child alpha_m1_link, origin xyz=0.02 0 0.033 rpy=0 0 2.09439, axis 0 0 -1, limit lower=0.0 upper=3.22 effort=9.0 velocity=0.5
- added joint alpha_axis_c: type revolute, parent alpha_m2_link, child alpha_m2_1_3_link, origin xyz=-0.04 0 -0.1453 rpy=0 0 3.14159, axis 0 1 0, limit lower=0.0 upper=3.22 effort=9.0 velocity=0.5
- added joint alpha_axis_d: type revolute, parent alpha_m2_1_1_link, child alpha_m2_link, origin xyz=-0.02 0 0.033, axis 0 1 0, limit lower=-3.49 upper=3.49 effort=9.0 velocity=0.5
- added joint alpha_axis_e: type revolute, parent alpha_m3_inline_link, child alpha_m2_1_1_link, origin xyz=0 0 0.014, axis 0 0 1, limit lower=0.0 upper=6.10 effort=9.0 velocity=0.5
- added joint alpha_base_joint: type fixed, parent mount_link, child alpha_base_link, origin xyz=0 0 0 rpy=0 0 0
- added joint alpha_mount_joint: type fixed, parent alpha_base_link, child alpha_m3_inline_link, origin xyz=0.124 0.004 0 rpy=0 0 0
- added joint alpha_rs1_130_joint: type revolute, parent alpha_rs1_124_link, child alpha_rs1_130_link, origin xyz=0 0.0155 0.0069 rpy=0 0 0, axis -1 0 0, limit lower=0 upper=0.5 effort=10 velocity=10, mimic joint=alpha_axis_a multiplier=51 offset=0
- added joint alpha_rs1_139_joint: type revolute, parent alpha_rs1_124_link, child alpha_rs1_139_link, origin xyz=0 -0.0155 0.0069 rpy=0 0 0, axis 1 0 0, limit lower=0 upper=0.5 effort=10 velocity=10, mimic joint=alpha_rs1_130_joint multiplier=1 offset=0
- added joint alpha_tcp_base_joint: type fixed, parent alpha_m1_link, child alpha_rs1_124_link, origin xyz=0 0 0.09975 rpy=0 0 0
- added joint alpha_tcp_joint: type fixed, parent alpha_rs1_124_link, child alpha_tcp, origin xyz=0 0 0.04 rpy=0 -1.5707963267948966 0
- added joint float_joint: type fixed, parent base_link, child float_link, origin xyz=0 0 0 rpy=0 0 0
- added joint mount_joint: type fixed, parent base_link, child mount_link, origin xyz=0.13 -0.109 0.029 rpy=0 0 0

Commit message: adding docs to thruster controllers

File: output.urdf (robot description, URDF)
Before this commit: robot uvms_pinocchio, 17 links, 16 joints
Links:
- added link thruster1, mass 0.002; visual mesh filename=file:///home/ubuntu/ws_blue/install/blue_description/share/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
- added link thruster2, mass 0.002; visual mesh filename=file:///home/ubuntu/ws_blue/install/blue_description/share/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
- added link thruster3, mass 0.002; visual mesh filename=file:///home/ubuntu/ws_blue/install/blue_description/share/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
- added link thruster4, mass 0.002; visual mesh filename=file:///home/ubuntu/ws_blue/install/blue_description/share/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
- added link thruster5, mass 0.002; visual mesh filename=file:///home/ubuntu/ws_blue/install/blue_description/share/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
- added link thruster6, mass 0.002; visual mesh filename=file:///home/ubuntu/ws_blue/install/blue_description/share/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
- added link thruster7, mass 0.002; visual mesh filename=file:///home/ubuntu/ws_blue/install/blue_description/share/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
- added link thruster8, mass 0.002; visual mesh filename=file:///home/ubuntu/ws_blue/install/blue_description/share/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
Joints:
- added joint thruster1_joint: type continuous, parent base_link, child thruster1, origin xyz=0.088 -0.102 -0.04 rpy=-1.571 1.571 -1.047, axis 0 0 -1
- added joint thruster2_joint: type continuous, parent base_link, child thruster2, origin xyz=0.088 0.102 -0.04 rpy=-1.571 1.571 -2.094, axis 0 0 -1
- added joint thruster3_joint: type continuous, parent base_link, child thruster3, origin xyz=-0.088 -0.102 -0.04 rpy=-1.571 1.571 1.047, axis 0 0 -1
- added joint thruster4_joint: type continuous, parent base_link, child thruster4, origin xyz=-0.088 0.102 -0.04 rpy=-1.571 1.571 2.094, axis 0 0 -1
- added joint thruster5_joint: type continuous, parent base_link, child thruster5, origin xyz=0.118 -0.215 0.064 rpy=0 0 0, axis 0 0 -1
- added joint thruster6_joint: type continuous, parent base_link, child thruster6, origin xyz=0.118 0.215 0.064 rpy=0 0 0, axis 0 0 -1
- added joint thruster7_joint: type continuous, parent base_link, child thruster7, origin xyz=-0.118 -0.215 0.064 rpy=0 0 0, axis 0 0 -1
- added joint thruster8_joint: type continuous, parent base_link, child thruster8, origin xyz=-0.118 0.215 0.064 rpy=0 0 0, axis 0 0 -1
